Commit message: 

File: description/robot_core.xacro (robot description, xacro)
@@ -1,4 +1,5 @@
 <?xml version="1.0"?>
 <robot xmlns:xacro="http://www.ros.org/wiki/xacro">
+    <xacro:include filename="inertial_macros.xacro"/>
   <!-- Materials -->
   <material name="white">
@@ -31,4 +32,14 @@
       <material name="white"/>
     </visual>
+        <collision>
+      <origin xyz="0.15 0 0.075"/>
+      <geometry>
+        <box size="0.3 0.3 0.15"/>
+      </geometry>
+      <material name="white"/>
+    </collision>
+    <xacro:inertial_box mass="0.5" x="0.3" y="0.3" z="0.15">
+      <origin xyz="0.15 0 0.075" rpy="0 0 0"/>
+    </xacro:inertial_box>
   </link>
   <!-- LEFT WHEEL LINK -->
@@ -46,4 +57,13 @@
       <material name="blue"/>
     </visual>
+        <collision>
+      <geometry>
+        <cylinder radius="0.05" length="0.04"/>
+      </geometry>
+      <material name="blue"/>
+    </collision>
+            <xacro:inertial_cylinder mass="0.1" length="0.04" radius="0.05">
+            <origin xyz="0 0 0" rpy="0 0 0"/>
+        </xacro:inertial_cylinder>
   </link>
   <!-- RIGHT WHEEL LINK -->
@@ -61,4 +81,36 @@
       <material name="blue"/>
     </visual>
+        <collision>
+      <geometry>
+        <cylinder radius="0.05" length="0.04"/>
+      </geometry>
+      <material name="blue"/>
+    </collision>
+            <xacro:inertial_cylinder mass="0.1" length="0.04" radius="0.05">
+            <origin xyz="0 0 0" rpy="0 0 0"/>
+        </xacro:inertial_cylinder>
+  </link>
+  <!-- Caster Wheel link -->
+  <joint name="caster_wheel_joint" type="fixed">
+    <parent link="base_link"/>
+    <child link="caster_wheel"/>
+    <origin xyz="0.24 0 0"/>
+  </joint>
+  <link name="caster_wheel">
+    <visual>
+        <geometry>
+          <sphere radius="0.05"/>
+      </geometry>
+      <material name="black"/>
+    </visual>
+        <collision>
+      <geometry>
+        <sphere radius="0.05"/>
+      </geometry>
+      <material name="black"/>
+    </collision>
+           <xacro:inertial_sphere mass="0.1" radius="0.05">
+            <origin xyz="0 0 0" rpy="0 0 0"/>
+        </xacro:inertial_sphere>
   </link>
 </robot>

File: install/my_bot/share/my_bot/description/robot_core.xacro (robot description, xacro)
@@ -1,4 +1,5 @@
 <?xml version="1.0"?>
 <robot xmlns:xacro="http://www.ros.org/wiki/xacro">
+    <xacro:include filename="inertial_macros.xacro"/>
   <!-- Materials -->
   <material name="white">
@@ -31,32 +32,85 @@
       <material name="white"/>
     </visual>
+        <collision>
+      <origin xyz="0.15 0 0.075"/>
+      <geometry>
+        <box size="0.3 0.3 0.15"/>
+      </geometry>
+      <material name="white"/>
+    </collision>
+    <xacro:inertial_box mass="0.5" x="0.3" y="0.3" z="0.15">
+      <origin xyz="0.15 0 0.075" rpy="0 0 0"/>
+    </xacro:inertial_box>
   </link>
-  <!-- LEFT WHEEL LINK-->
+  <!-- LEFT WHEEL LINK -->
   <joint name="left_wheel_joint" type="continuous">
     <parent link="base_link"/>
     <child link="left_wheel"/>
-    <origin xyz="0 0.175 0" rpy="-${pi/2 0 0}"/><!-- -${pi/2 0 0}-->
+    <origin xyz="0 0.175 0" rpy="-${pi/2} 0 0"/>
     <axis xyz="0 0 1"/>
   </joint>
   <link name="left_wheel">
-  <visual>
-  <geometry>
-    <cylinder radius="0.05" length="0.04"/>
-  </geometry>
-  <material name="blue"/>
+    <visual>
+      <geometry>
+        <cylinder radius="0.05" length="0.04"/>
+      </geometry>
+      <material name="blue"/>
+    </visual>
+        <collision>
+      <geometry>
+        <cylinder radius="0.05" length="0.04"/>
+      </geometry>
+      <material name="blue"/>
+    </collision>
+            <xacro:inertial_cylinder mass="0.1" length="0.04" radius="0.05">
+            <origin xyz="0 0 0" rpy="0 0 0"/>
+        </xacro:inertial_cylinder>
   </link>
-  <!-- RIGHT WHEEL LINK-->
+  <!-- RIGHT WHEEL LINK -->
   <joint name="right_wheel_joint" type="continuous">
     <parent link="base_link"/>
     <child link="right_wheel"/>
-    <origin xyz="0 -0.175 0" rpy="${pi/2 0 0}"/><!-- -${pi/2 0 0}-->
+    <origin xyz="0 -0.175 0" rpy="${pi/2} 0 0"/>
     <axis xyz="0 0 -1"/>
   </joint>
   <link name="right_wheel">
-  <visual>
-  <geometry>
-    <cylinder radius="0.05" length="0.04"/>
-  </geometry>
-  <material name="blue"/>
+    <visual>
+      <geometry>
+        <cylinder radius="0.05" length="0.04"/>
+      </geometry>
+      <material name="blue"/>
+    </visual>
+        <collision>
+      <geometry>
+        <cylinder radius="0.05" length="0.04"/>
+      </geometry>
+      <material name="blue"/>
+    </collision>
+            <xacro:inertial_cylinder mass="0.1" length="0.04" radius="0.05">
+            <origin xyz="0 0 0" rpy="0 0 0"/>
+        </xacro:inertial_cylinder>
+  </link>
+  <!-- Caster Wheel link -->
+  <joint name="caster_wheel_joint" type="fixed">
+    <parent link="base_link"/>
+    <child link="caster_wheel"/>
+    <origin xyz="0.24 0 0"/>
+  </joint>
+  <link name="caster_wheel">
+    <visual>
+        <geometry>
+          <sphere radius="0.05"/>
+      </geometry>
+      <material name="black"/>
+    </visual>
+        <collision>
+      <geometry>
+        <sphere radius="0.05"/>
+      </geometry>
+      <material name="black"/>
+    </collision>
+           <xacro:inertial_sphere mass="0.1" radius="0.05">
+            <origin xyz="0 0 0" rpy="0 0 0"/>
+        </xacro:inertial_sphere>
   </link>
 </robot>
